File: ICE40-DIO_Rev_A.kicad_pcb (KiCad board)
At the start: 2 copper layers, 50 x 50 mm, 51 parts, among them U1 MCP47A1T-A0E/LT(SC70-6), U2 74ALVC164245DL(SSOP48), U3 74ALVC164245DL(SSOP48)

Commit message: Update
Changed trace names
Connections:
- net /LED1 renamed /GPIO_Pin<10>
- net /LED2 renamed /GPIO_Pin<12>
- net /PIO2_1 renamed /GPIO_Pin<30>
- net /PIO2_2 renamed /UEXT_#SS
- net /PIO2_3 renamed /UEXT_SCK
- net /PIO2_4 renamed /UEXT_MOSI
- net /PIO2_5 renamed /UEXT_MISO
- net /PIO2_6 renamed /UEXT_SDA
- net /PIO2_7 renamed /UEXT_SCL
- net /PIO2_8/TxD renamed /UEXT_TxD
- net /PIO2_9/RxD renamed /UEXT_RxD
- net /PIO3_10A renamed /GPIO_Pin<31>
- net /PIO3_10B renamed /GPIO_Pin<33>
- net /PIO3_12A renamed /GPIO_Pin<34>
- net /PIO3_12B renamed /GPIO_Pin<32>
- net /PIO3_1A renamed /GPIO_Pin<5>
- net /PIO3_1B renamed /GPIO_Pin<7>
- net /PIO3_2A renamed /GPIO_Pin<9>
- net /PIO3_2B renamed /GPIO_Pin<11>
- net /PIO3_3A renamed /GPIO_Pin<13>
- net /PIO3_3B renamed /GPIO_Pin<15>
- net /PIO3_5A renamed /GPIO_Pin<17>
- net /PIO3_5B renamed /GPIO_Pin<19>
- net /PIO3_6A renamed /GPIO_Pin<21>
- net /PIO3_6B renamed /GPIO_Pin<23>
- net /PIO3_7B renamed /GPIO_Pin<25>
- net /PIO3_8A renamed /GPIO_Pin<27>
- net /PIO3_8B renamed /GPIO_Pin<29>
- U3 pad 19: (no net) -> Net-(U3-Pad19)
- U3 pad 20: (no net) -> Net-(U3-Pad20)
- U3 pad 22: (no net) -> Net-(U3-Pad22)
- U3 pad 23: (no net) -> Net-(U3-Pad23)
- U3 pad 26: (no net) -> Net-(U3-Pad26)
- U3 pad 27: (no net) -> Net-(U3-Pad27)
- U3 pad 29: (no net) -> Net-(U3-Pad29)
- U3 pad 30: (no net) -> Net-(U3-Pad30)
